File: schematic/sub_rf_mod.kicad_sch (KiCad schematic)
At the start: 72 parts, among them J1 Conn_01x08, J2 MD-90SM, Q1 2N3906, U1 NE5532, U2 MAX4395ESD, U3 LM1881, U5 ADG453, U6 LMH1251, U7 MAX4395ESD, U8 L7805

Commit message: add schematic
Parts:
- added L1: 4.7uH, Inductor_THT:L_Axial_L7.0mm_D3.3mm_P10.16mm_Horizontal_Fastron_MICC, symbol Device:L
Connections:
- net +5VD: now also L1.2; no longer R2.2, R26.2
- net +5VA: now reaches C2.2, R26.1, U1.8 (V+)
- net +5VA: now also R2.2
- new net: L1.1, R26.2
Other:
- moved on the sheet: C2, R26, U1C
